File: MPCNC Mega 2560 Pro.brd (EAGLE design)
At the start: 160 x 100 mm, 193 parts, among them IC1 MEGA2560-PRO, IC10 SFH6156, IC11 SFH6156, IC12 SFH6156, IC13 SFH6156, IC14 SFH6156, IC15 SFH6156, IC16 SFH6156, IC17 SFH6156, IC18 SFH6156, IC19 SFH6156, IC2 ULN2003AD, IC20 SFH6156, IC21 SFH6156, IC3 ULN2003AD, IC4 SFH6156, IC5 LM358D, IC6 SFH6156, IC7 SFH6156, IC8 SFH6156, IC9 SFH6156, J1 22-27-2031-03, J11 VFD On/Off, J12 VFD 0-10V, J2 22-27-2031-03, J3 22-27-2031-03, J4 Stepper Enable, J9 Out Spindle, U1 TSR2-24120, U2 TSR2-2450, X1 MSTBV2, X2 22-27-2031-03, X3 22-27-2031-03

Commit message: Added readme and license, Added license information in circuit
Other:
- board text added: "CC BY-NC-SA 4.0 Peter Müller peter@crycode.de"
- board text removed: "(CC) BY-NC-SA 4.0 Peter Müller peter@crycode.de"
Changed lines of the file:
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@@
 <text x="68.58" y="66.04" size="1.016" layer="25" font="vector" ratio="20" align="top-center">Analog IN</text>
 <wire x1="149.86" y1="71.12" x2="160" y2="71.12" width="0.3048" layer="21" style="shortdash"/>
-<text x="88.265" y="24.13" size="1.016" layer="21" font="vector" ratio="15" rot="R90" align="top-center">(CC) BY-NC-SA 4.0
+<text x="88.265" y="24.13" size="1.016" layer="21" font="vector" ratio="15" rot="R90" align="top-center">CC BY-NC-SA 4.0
 Peter Müller
 peter@crycode.de</text>

Commit message: Added reset connector, Fixed multiline information in circuit
Parts:
- added J5: 22-27-2021-02, con-molex:6410-02
Connections:
- new net !RESET: IC1.RST, J5.1
- net GND: now also J5.2
Routing:
- net !RESET: track 0.00 -> 8.25 mm
- net SPINDLE_SPEED_PWM: track 30.5 -> 32.0 mm
- net OUT_COM: track 192.3 -> 191.6 mm
- net OUT_8: track 95.5 -> 94.8 mm
Other:
- board text added: "Reset"
