File: MPCNC Mega 2560 Pro.brd (EAGLE design)
At the start: 160 x 100 mm, 194 parts, among them IC1 MEGA2560-PRO, IC10 SFH6156, IC11 SFH6156, IC12 SFH6156, IC13 SFH6156, IC14 SFH6156, IC15 SFH6156, IC16 SFH6156, IC17 SFH6156, IC18 SFH6156, IC19 SFH6156, IC2 ULN2003AD, IC20 SFH6156, IC21 SFH6156, IC3 ULN2003AD, IC4 SFH6156, IC5 LM358D, IC6 SFH6156, IC7 SFH6156, IC8 SFH6156, IC9 SFH6156, J1 22-27-2031-03, J11 VFD On/Off, J12 VFD 0-10V, J2 22-27-2031-03, J3 22-27-2031-03, J4 Stepper Enable, J5 22-27-2021-02, J9 Out Spindle, U1 TSR2-24120, U2 TSR2-2450, X1 MSTBV2, X2 22-27-2031-03, X3 22-27-2031-03

Commit message: Switched to low current LEDs
Parts:
- LED1, LED2, LED3: value (none) -> 2mA, bl
- LED10, LED11, LED12, LED13, LED14, LED15, LED16, LED17, LED18, LED19, LED20, LED21, LED22, LED23, LED24, LED25, LED26, LED27, LED28, LED4, LED5, LED6, LED7, LED8, LED9: value 25 mA 3,2V bl -> 2mA, bl
- R1: value (none) -> 22k
- R10, R11, R12, R13, R14, R15, R16, R17, R34, R35, R36, R37, R38, R39, R40, R41, R42, R43, R44, R45, R46, R47, R48, R49, R9: value 120 -> 1k2
- R7: value (none) -> 4k7
- R8: value (none) -> 1k2

Commit message: Fixed resistor value
Parts:
- R6: value 1k -> 1k2
Changed lines of the file:
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@@
 <attribute name="VALUE" x="133.096" y="12.065" size="1.27" layer="27" ratio="10" rot="R90"/>
 </element>
-<element name="R6" library="rcl" package="R1206" value="1k" x="133.35" y="7.62" smashed="yes" rot="R270">
+<element name="R6" library="rcl" package="R1206" value="1k2" x="133.35" y="7.62" smashed="yes" rot="R270">
 <attribute name="NAME" x="133.35" y="10.16" size="0.8128" layer="25" font="vector" rot="R90" align="center-left"/>
 <attribute name="VALUE" x="130.81" y="8.89" size="1.27" layer="27" rot="R270"/>

Commit message: V1.2 Rev. 4, Fixed issue #1
Pin 2 and 3 of IC5 were swapped
Thanks to @Gerssi for reporting!
Connections:
- net N$66: now also IC5.2; no longer IC5.3
- net N$71: now also IC5.3; no longer IC5.2
Routing:
- net N$66: track 14.9 -> 13.7 mm
- net N$71: track 13.1 -> 12.6 mm
Other:
- board text added: "MPCNC Mega 2560 Pro Shield v1.2 Rev. 4"
- board text removed: "MPCNC Mega 2560 Pro Shield"
- board text removed: "MPCNC Mega 2560 Pro Shield v1.2"
Changed lines of the file:
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@@
 <?xml version="1.0" encoding="utf-8"?>
 <!DOCTYPE eagle SYSTEM "eagle.dtd">
-<eagle version="7.4.0">
+<eagle version="7.7.0">
 <drawing>
 <settings>
@@
 <setting verticaltext="up"/>
 </settings>
-<grid distance="0.05" unitdist="inch" unit="mm" style="lines" multiple="1" display="yes" altdistance="0.0125" altunitdist="inch" altunit="inch"/>
+<grid distance="0.05" unitdist="inch" unit="mm" style="lines" multiple="1" display="no" altdistance="0.0125" altunitdist="inch" altunit="inch"/>
 <layers>
 <layer number="1" name="Top" color="4" fill="1" visible="yes" active="yes"/>
@@
 <vertex x="47.625" y="21.2725" curve="-90"/>
 </polygon>
-<text x="95.25" y="69.215" size="1.778" layer="25" font="vector" ratio="20" align="center">MPCNC Mega 2560 Pro Shield v1.2</text>
+<text x="100.33" y="69.215" size="1.778" layer="25" font="vector" ratio="20" align="center">MPCNC Mega 2560 Pro Shield v1.2 Rev. 4</text>
 <text x="107.95" y="2.54" size="1.016" layer="25" font="vector" ratio="15" align="bottom-right">Mega 2560 Pro</text>
 <wire x1="35.95" y1="100" x2="35.95" y2="85.725" width="0.3048" layer="21" style="shortdash"/>
@@
 Peter Müller
 peter@crycode.de</text>
-<text x="93.98" y="80.01" size="1.778" layer="16" font="vector" ratio="20" rot="MR0" align="center">MPCNC Mega 2560 Pro Shield</text>
+<text x="93.98" y="80.01" size="1.778" layer="16" font="vector" ratio="20" rot="MR0" align="center">MPCNC Mega 2560 Pro Shield v1.2 Rev. 4</text>
 <text x="31.75" y="98.1075" size="1.016" layer="25" font="vector" ratio="15" align="bottom-center">15-36V</text>
 <text x="26.9875" y="86.36" size="1.27" layer="25" font="vector" ratio="15" align="bottom-right">-</text>
@@
 </signal>
 <signal name="N$66">
-<contactref element="IC5" pad="3"/>
 <contactref element="R4" pad="2"/>
 <contactref element="JP9" pad="2"/>
-<wire x1="136.525" y1="9.585" x2="136.525" y2="8.255" width="0.4064" layer="1"/>
-<wire x1="136.525" y1="8.255" x2="137.16" y2="7.62" width="0.4064" layer="1"/>
-<wire x1="137.16" y1="7.62" x2="142.875" y2="7.62" width="0.4064" layer="1"/>
+<wire x1="137.795" y1="8.255" x2="138.43" y2="7.62" width="0.4064" layer="1"/>
+<wire x1="138.43" y1="7.62" x2="142.875" y2="7.62" width="0.4064" layer="1"/>
 <wire x1="142.875" y1="7.62" x2="148.59" y2="7.62" width="0.4064" layer="1"/>
 <wire x1="142.875" y1="8.89" x2="142.875" y2="7.62" width="0.4064" layer="1"/>
+<contactref element="IC5" pad="2"/>
+<wire x1="137.795" y1="8.255" x2="137.795" y2="9.585" width="0.4064" layer="1"/>
 </signal>
 <signal name="N$67">
@@
 <signal name="N$71">
 <contactref element="C8" pad="+"/>
-<contactref element="IC5" pad="2"/>
 <contactref element="R6" pad="1"/>
 <contactref element="JP7" pad="1"/>
@@
 <wire x1="133.198" y1="8.89" x2="133.35" y2="9.042" width="0.4064" layer="1"/>
 <wire x1="133.35" y1="9.042" x2="133.35" y2="10.795" width="0.4064" layer="1"/>
-<wire x1="137.795" y1="9.585" x2="137.795" y2="11.43" width="0.4064" layer="1"/>
-<wire x1="137.795" y1="11.43" x2="135.89" y2="13.335" width="0.4064" layer="1"/>
 <wire x1="133.35" y1="10.795" x2="135.89" y2="13.335" width="0.4064" layer="1"/>
+<contactref element="IC5" pad="3"/>
+<wire x1="136.525" y1="9.585" x2="136.525" y2="12.7" width="0.4064" layer="1"/>
+<wire x1="136.525" y1="12.7" x2="135.89" y2="13.335" width="0.4064" layer="1"/>
 </signal>
 <signal name="N$75">
