File: MPCNC Mega 2560 Pro.sch (EAGLE design)
At the start: 192 parts, among them IC1 MEGA2560-PRO, IC10 SFH6156, IC11 SFH6156, IC12 SFH6156, IC13 SFH6156, IC14 SFH6156, IC15 SFH6156, IC16 SFH6156, IC17 SFH6156, IC18 SFH6156, IC19 SFH6156, IC2 ULN2003AD, IC20 SFH6156, IC21 SFH6156, IC3 ULN2003AD, IC4 SFH6156, IC5 LM358D, IC6 SFH6156, IC7 SFH6156, IC8 SFH6156, IC9 SFH6156, J1 22-27-2031-03, J11 VFD On/Off, J12 VFD 0-10V, J2 22-27-2031-03, J3 22-27-2031-03, J4 Stepper Enable, J9 Out Spindle, U1 TSR2-24120, U2 TSR2-2450, X1 MSTBV2, X2 22-27-2031-03, X3 22-27-2031-03

Commit message: Added readme and license, Added license information in circuit
Other:
- note added: "Sheet:"
- note added: "Solder pads for currently unused pins"
- note removed: "LEDs: RND 135-00183 (SMD, 0805, blau, 160 mcd)"
- note removed: "Solder pads for remaining pins"
Changed lines of the file:
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@@
 <schematic xreflabel="%F%N/%S.%C%R" xrefpart="/%S.%C%R">
 <attributes>
+<attribute name="BASED_ON" value="Parts based on MPCNC Nano Estlcam
+ Shield by Till Nenz"/>
+<attribute name="BY" value="Created and Copyright by
+ Peter Müller &lt;peter@crycode.de&gt;,
+ Günter Brauer &lt;gbzzr1100@gmail.de&gt;"/>
+<attribute name="DOC_NAME" value="MPCNC Mega 2560 Pro Shield"/>
+<attribute name="LICENSE" value="Creative Commons CC-BY-SA-NC 4.0 License"/>
+<attribute name="VERSION" value="v1.2"/>
 </attributes>
 <variantdefs>
@@
 <part name="MS-X1" library="jumper" deviceset="JP3Q" device=""/>
 <part name="C1" library="rcl" deviceset="CPOL-EU" device="E2.5-7" value="100 µF"/>
-<part name="FRAME1" library="frames" deviceset="A4L-LOC" device=""/>
-<part name="FRAME2" library="frames" deviceset="A4L-LOC" device=""/>
+<part name="FRAME1" library="frames" deviceset="A4L-LOC-NO-NAMES" device=""/>
+<part name="FRAME2" library="frames" deviceset="A4L-LOC-NO-NAMES" device=""/>
 <part name="S.DRIVER-X2" library="stepper-driver" deviceset="STEPPER-DRIVER" device=""/>
 <part name="MS-X2" library="jumper" deviceset="JP3Q" device=""/>
@@
 <part name="U1" library="TSR" deviceset="TSR2-*" device="" technology="24120"/>
 <part name="U2" library="TSR" deviceset="TSR2-*" device="" technology="2450"/>
-<part name="FRAME3" library="frames" deviceset="A4L-LOC" device=""/>
+<part name="FRAME3" library="frames" deviceset="A4L-LOC-NO-NAMES" device=""/>
 <part name="X1" library="con-phoenix-508" deviceset="MSTBV2" device=""/>
 <part name="IC1" library="mega2560-pro-mini" deviceset="MEGA2560-PRO" device=""/>
@@
 <part name="R1" library="rcl" deviceset="R-EU_" device="R1206"/>
 <part name="C7" library="rcl" deviceset="CPOL-EU" device="E2-5" value="22 µF / 50 V Low ESR"/>
-<part name="FRAME5" library="frames" deviceset="A4L-LOC" device=""/>
+<part name="FRAME5" library="frames" deviceset="A4L-LOC-NO-NAMES" device=""/>
 <part name="IC2" library="uln-udn" deviceset="ULN2003A" device="D"/>
 <part name="IC3" library="uln-udn" deviceset="ULN2003A" device="D"/>
@@
 <part name="IN15" library="con-molex" deviceset="22-?-03" device="27-2031" value="22-27-2031-03"/>
 <part name="IN16" library="con-molex" deviceset="22-?-03" device="27-2031" value="22-27-2031-03"/>
-<part name="FRAME7" library="frames" deviceset="A4L-LOC" device=""/>
+<part name="FRAME7" library="frames" deviceset="A4L-LOC-NO-NAMES" device=""/>
 <part name="IC6" library="optocoupler" deviceset="SFH6156" device=""/>
 <part name="R18" library="rcl" deviceset="R-EU_" device="R1206" value="220"/>
@@
 <part name="X2" library="con-molex" deviceset="22-?-03" device="27-2031"/>
 <part name="X3" library="con-molex" deviceset="22-?-03" device="27-2031"/>
-<part name="FRAME8" library="frames" deviceset="A4L-LOC" device=""/>
+<part name="FRAME8" library="frames" deviceset="A4L-LOC-NO-NAMES" device=""/>
 <part name="R34" library="rcl" deviceset="R-EU_" device="R1206" value="120"/>
 <part name="LED13" library="led" deviceset="LED" device="CHIPLED_0805" value="25 mA 3,2V bl"/>
@@
 <text x="7.62" y="170.18" size="1.778" layer="97">Mega 2560 Pro Board</text>
 <wire x1="134.62" y1="38.1" x2="4.318" y2="38.1" width="0.6096" layer="97" style="shortdash"/>
-<text x="7.62" y="33.02" size="1.778" layer="97">Solder pads for remaining pins</text>
+<text x="7.62" y="33.02" size="1.778" layer="97">Solder pads for currently unused pins</text>
+<text x="162.56" y="22.86" size="1.778" layer="94" align="top-left">&gt;LICENSE</text>
+<text x="215.9" y="22.86" size="1.778" layer="94" ratio="10" align="top-left">&gt;DOC_NAME</text>
+<text x="215.9" y="17.78" size="1.778" layer="94" ratio="10" align="top-left">&gt;VERSION</text>
+<text x="215.9" y="7.62" size="1.778" layer="94" ratio="10" align="top-left">Sheet:</text>
+<text x="254" y="7.62" size="1.778" layer="94" ratio="10" align="top-right">&gt;SHEET</text>
+<text x="162.56" y="19.05" size="1.778" layer="94" align="top-left">&gt;BY</text>
+<text x="162.56" y="10.16" size="1.778" layer="94" align="top-left">&gt;BASED_ON</text>
 </plain>
 <instances>
@@
 <text x="91.44" y="99.06" size="1.778" layer="97">+5V / +12V / GND Connectors</text>
 <text x="180.34" y="99.06" size="1.778" layer="97">Fan Connector</text>
+<text x="162.56" y="22.86" size="1.778" layer="94" align="top-left">&gt;LICENSE</text>
+<text x="215.9" y="22.86" size="1.778" layer="94" ratio="10" align="top-left">&gt;DOC_NAME</text>
+<text x="215.9" y="17.78" size="1.778" layer="94" ratio="10" align="top-left">&gt;VERSION</text>
+<text x="215.9" y="7.62" size="1.778" layer="94" ratio="10" align="top-left">Sheet:</text>
+<text x="254" y="7.62" size="1.778" layer="94" ratio="10" align="top-right">&gt;SHEET</text>
+<text x="162.56" y="19.05" size="1.778" layer="94" align="top-left">&gt;BY</text>
+<text x="162.56" y="10.16" size="1.778" layer="94" align="top-left">&gt;BASED_ON</text>
 </plain>
 <instances>
@@
 <text x="7.62" y="55.88" size="1.778" layer="97">Stepper Driver Z</text>
 <text x="134.62" y="55.88" size="1.778" layer="97">External Stepper Driver Connectors</text>
+<text x="162.56" y="22.86" size="1.778" layer="94" align="top-left">&gt;LICENSE</text>
+<text x="215.9" y="22.86" size="1.778" layer="94" ratio="10" align="top-left">&gt;DOC_NAME</text>
+<text x="215.9" y="17.78" size="1.778" layer="94" ratio="10" align="top-left">&gt;VERSION</text>
+<text x="215.9" y="7.62" size="1.778" layer="94" ratio="10" align="top-left">Sheet:</text>
+<text x="254" y="7.62" size="1.778" layer="94" ratio="10" align="top-right">&gt;SHEET</text>
+<text x="162.56" y="19.05" size="1.778" layer="94" align="top-left">&gt;BY</text>
+<text x="162.56" y="10.16" size="1.778" layer="94" align="top-left">&gt;BASED_ON</text>
 </plain>
 <instances>
@@
 <description>Digital Out</description>
 <plain>
-<text x="162.56" y="7.62" size="1.778" layer="97" align="top-left">* VFD = Variable Frequency Drive</text>
+<text x="114.3" y="7.62" size="1.778" layer="97" align="top-left">* VFD = Variable Frequency Drive</text>
 <wire x1="256.032" y1="119.38" x2="154.94" y2="119.38" width="0.6096" layer="97" style="shortdash"/>
 <wire x1="81.28" y1="132.08" x2="1.778" y2="132.08" width="0.6096" layer="97" style="shortdash"/>
@@
 <text x="157.48" y="170.18" size="1.778" layer="97">Output Status LEDs</text>
 <text x="7.62" y="170.18" size="1.778" layer="97">Output Drivers</text>
+<text x="162.56" y="22.86" size="1.778" layer="94" align="top-left">&gt;LICENSE</text>
+<text x="215.9" y="22.86" size="1.778" layer="94" ratio="10" align="top-left">&gt;DOC_NAME</text>
+<text x="215.9" y="17.78" size="1.778" layer="94" ratio="10" align="top-left">&gt;VERSION</text>
+<text x="215.9" y="7.62" size="1.778" layer="94" ratio="10" align="top-left">Sheet:</text>
+<text x="254" y="7.62" size="1.778" layer="94" ratio="10" align="top-right">&gt;SHEET</text>
+<text x="162.56" y="19.05" size="1.778" layer="94" align="top-left">&gt;BY</text>
+<text x="162.56" y="10.16" size="1.778" layer="94" align="top-left">&gt;BASED_ON</text>
 </plain>
 <instances>
@@
 <description>Digital In</description>
 <plain>
-<text x="162.56" y="22.86" size="1.778" layer="97" align="top-left">LEDs:
-RND 135-00183 (SMD, 0805, blau, 160 mcd)</text>
 <wire x1="165.1" y1="24.638" x2="165.1" y2="174.752" width="0.6096" layer="97" style="shortdash"/>
 <text x="7.62" y="170.18" size="1.778" layer="97">Digital Inputs (via Optocouplers)</text>
 <text x="170.18" y="170.18" size="1.778" layer="97">Digital Input Status LEDs</text>
+<text x="162.56" y="22.86" size="1.778" layer="94" align="top-left">&gt;LICENSE</text>
+<text x="215.9" y="22.86" size="1.778" layer="94" ratio="10" align="top-left">&gt;DOC_NAME</text>
+<text x="215.9" y="17.78" size="1.778" layer="94" ratio="10" align="top-left">&gt;VERSION</text>
+<text x="215.9" y="7.62" size="1.778" layer="94" ratio="10" align="top-left">Sheet:</text>
+<text x="254" y="7.62" size="1.778" layer="94" ratio="10" align="top-right">&gt;SHEET</text>
+<text x="162.56" y="19.05" size="1.778" layer="94" align="top-left">&gt;BY</text>
+<text x="162.56" y="10.16" size="1.778" layer="94" align="top-left">&gt;BASED_ON</text>
 </plain>
 <instances>
@@
 <plain>
 <text x="7.62" y="170.18" size="1.778" layer="97">Digital In Connectors</text>
+<text x="162.56" y="22.86" size="1.778" layer="94" align="top-left">&gt;LICENSE</text>
+<text x="215.9" y="22.86" size="1.778" layer="94" ratio="10" align="top-left">&gt;DOC_NAME</text>
+<text x="215.9" y="17.78" size="1.778" layer="94" ratio="10" align="top-left">&gt;VERSION</text>
+<text x="215.9" y="7.62" size="1.778" layer="94" ratio="10" align="top-left">Sheet:</text>
+<text x="254" y="7.62" size="1.778" layer="94" ratio="10" align="top-right">&gt;SHEET</text>
+<text x="162.56" y="19.05" size="1.778" layer="94" align="top-left">&gt;BY</text>
+<text x="162.56" y="10.16" size="1.778" layer="94" align="top-left">&gt;BASED_ON</text>
 </plain>
 <instances>
@@
 </schematic>
 </drawing>
-<compatibility>
-<note version="6.3" minversion="6.2.2" severity="warning">
-Since Version 6.2.2 text objects can contain more than one line,
-which will not be processed correctly with this version.
-</note>
-</compatibility>
 </eagle>

Commit message: Added reset connector, Fixed multiline information in circuit
Parts:
- added J5: 22-27-2021-02, con-molex:22-27-2021-02
Connections:
- new net !RESET: IC1.!RESET, J5-1.S
- net GND: now also J5-2.S
Other:
- note added: "External Reset"
- moved on the sheet: SV1

Commit message: Switched to low current LEDs
Parts:
- LED1, LED2, LED3: value (none) -> 2mA, bl
- LED10, LED11, LED12, LED13, LED14, LED15, LED16, LED17, LED18, LED19, LED20, LED21, LED22, LED23, LED24, LED25, LED26, LED27, LED28, LED4, LED5, LED6, LED7, LED8, LED9: value 25 mA 3,2V bl -> 2mA, bl
- R1: value (none) -> 22k
- R10, R11, R12, R13, R14, R15, R16, R17, R34, R35, R36, R37, R38, R39, R40, R41, R42, R43, R44, R45, R46, R47, R48, R49, R9: value 120 -> 1k2
- R7: value (none) -> 4k7
- R8: value (none) -> 1k2

Commit message: Fixed resistor value
Parts:
- R6: value 1k -> 1k2
Changed lines of the file:
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@@
 <part name="JP7" library="jumper" deviceset="JP1Q" device="" value="PWM"/>
 <part name="JP8" library="jumper" deviceset="JP1Q" device="" value="Analog"/>
-<part name="R6" library="rcl" deviceset="R-EU_" device="R1206" value="1k"/>
+<part name="R6" library="rcl" deviceset="R-EU_" device="R1206" value="1k2"/>
 <part name="JP9" library="jumper" deviceset="JP1Q" device="" value="5V / 10V"/>
 <part name="LED2" library="led" deviceset="LED" device="CHIPLED_1206" value="2mA, bl"/>

Commit message: V1.2 Rev. 4, Fixed issue #1
Pin 2 and 3 of IC5 were swapped
Thanks to @Gerssi for reporting!
Connections:
- net N$66: now also IC5A.-IN; no longer IC5A.+IN
- net N$71: now also IC5A.+IN; no longer IC5A.-IN
Other:
- moved on the sheet: IC5A
Changed lines of the file:
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@@
 <?xml version="1.0" encoding="utf-8"?>
 <!DOCTYPE eagle SYSTEM "eagle.dtd">
-<eagle version="7.4.0">
+<eagle version="7.7.0">
 <drawing>
 <settings>
@@
 <attribute name="DOC_NAME" value="MPCNC Mega 2560 Pro Shield"/>
 <attribute name="LICENSE" value="Creative Commons CC-BY-SA-NC 4.0 License"/>
-<attribute name="VERSION" value="v1.2 Rev. 3"/>
+<attribute name="VERSION" value="v1.2 Rev. 4"/>
 </attributes>
 <variantdefs>
@@
 <instance part="J11" gate="-1" x="58.42" y="96.52"/>
 <instance part="J11" gate="-2" x="58.42" y="91.44"/>
-<instance part="IC5" gate="A" x="55.88" y="43.18" rot="R180"/>
-<instance part="IC5" gate="P" x="55.88" y="43.18"/>
+<instance part="IC5" gate="A" x="55.88" y="48.26" rot="R180"/>
+<instance part="IC5" gate="P" x="55.88" y="48.26"/>
 <instance part="J12" gate="-1" x="17.78" y="30.48" rot="MR0"/>
 <instance part="J12" gate="-2" x="17.78" y="25.4" rot="MR0"/>
@@
 <segment>
 <pinref part="IC5" gate="P" pin="V+"/>
-<wire x1="55.88" y1="50.8" x2="55.88" y2="53.34" width="0.1524" layer="91"/>
-<label x="55.88" y="53.34" size="1.778" layer="95"/>
+<wire x1="55.88" y1="55.88" x2="55.88" y2="58.42" width="0.1524" layer="91"/>
+<label x="55.88" y="58.42" size="1.778" layer="95"/>
 </segment>
 </net>
@@
 <segment>
 <pinref part="IC5" gate="P" pin="V-"/>
-<wire x1="55.88" y1="35.56" x2="55.88" y2="7.62" width="0.1524" layer="91"/>
+<wire x1="55.88" y1="40.64" x2="55.88" y2="7.62" width="0.1524" layer="91"/>
 <pinref part="R5" gate="G$1" pin="2"/>
 <wire x1="83.82" y1="15.24" x2="81.28" y2="15.24" width="0.1524" layer="91"/>
@@
 <net name="N$66" class="0">
 <segment>
-<pinref part="IC5" gate="A" pin="+IN"/>
 <pinref part="R4" gate="G$1" pin="S"/>
-<wire x1="63.5" y1="40.64" x2="63.5" y2="30.48" width="0.1524" layer="91"/>
 <pinref part="JP9" gate="A" pin="2"/>
 <wire x1="63.5" y1="30.48" x2="63.5" y2="20.32" width="0.1524" layer="91"/>
 <wire x1="53.34" y1="30.48" x2="63.5" y2="30.48" width="0.1524" layer="91"/>
+<pinref part="IC5" gate="A" pin="-IN"/>
+<wire x1="63.5" y1="50.8" x2="66.04" y2="50.8" width="0.1524" layer="91"/>
+<wire x1="66.04" y1="50.8" x2="66.04" y2="30.48" width="0.1524" layer="91"/>
+<wire x1="66.04" y1="30.48" x2="63.5" y2="30.48" width="0.1524" layer="91"/>
 <junction x="63.5" y="30.48"/>
 </segment>
@@
 <wire x1="35.56" y1="15.24" x2="35.56" y2="30.48" width="0.1524" layer="91"/>
 <pinref part="IC5" gate="A" pin="OUT"/>
-<wire x1="35.56" y1="30.48" x2="35.56" y2="43.18" width="0.1524" layer="91"/>
-<wire x1="35.56" y1="43.18" x2="48.26" y2="43.18" width="0.1524" layer="91"/>
+<wire x1="35.56" y1="30.48" x2="35.56" y2="48.26" width="0.1524" layer="91"/>
+<wire x1="35.56" y1="48.26" x2="48.26" y2="48.26" width="0.1524" layer="91"/>
 <pinref part="J12" gate="-1" pin="S"/>
 <wire x1="20.32" y1="30.48" x2="35.56" y2="30.48" width="0.1524" layer="91"/>
@@
 <pinref part="C8" gate="G$1" pin="+"/>
 <wire x1="83.82" y1="43.18" x2="83.82" y2="45.72" width="0.1524" layer="91"/>
-<pinref part="IC5" gate="A" pin="-IN"/>
-<wire x1="83.82" y1="45.72" x2="63.5" y2="45.72" width="0.1524" layer="91"/>
 <pinref part="R6" gate="G$1" pin="1"/>
 <wire x1="88.9" y1="45.72" x2="83.82" y2="45.72" width="0.1524" layer="91"/>
@@
 <pinref part="JP7" gate="A" pin="1"/>
 <wire x1="83.82" y1="55.88" x2="86.36" y2="55.88" width="0.1524" layer="91"/>
-</segment>
-</net>
+<pinref part="IC5" gate="A" pin="+IN"/>
+<wire x1="63.5" y1="45.72" x2="83.82" y2="45.72" width="0.1524" layer="91"/>
+</segment>
+</net>
